Commit message: sync with diffcontrol repo

File: urdf/arm.urdf (robot description, URDF)
Before this commit: robot omnipointer, 7 links, 6 joints
Links:
- link arm_link_0: mass 0.2 -> 100.2
- link base_link: mass 0.0 -> 0.1
Joints:
- joint arm_joint_0: origin xyz=0 0 0 rpy=0 0 0 -> xyz=0 0 0.8 rpy=0 0 0
- joint arm_joint_1: axis 0 0 1 -> 0 1 0

File: urdf/cartpole_add_base.urdf (robot description, URDF)
Before this commit: robot physics, 3 links, 2 joints
Links:
- added link base_link, mass 0.1
- link pole: mass 0.5 -> 0.1; geometry collision box size=0.05 0.05 1.0; visual box size=0.08 0.08 1.0
- link slideBar: mass 1.0 -> 10000.
Joints:
- added joint base_to_slide: type fixed, parent base_link, child slideBar, origin xyz=0 0 1.0 rpy=0 0 0
- joint cart_to_pole: limit lower=-1.5 upper=1.5 effort=30.0 velocity=5.0 -> lower=-3.1415926535 upper=3.1415926535 effort=30.0 velocity=100.0
