Commit message: update simulator

File: urdf/quadrupedal.urdf (robot description, URDF)
Before this commit: robot quadruped_test, 3 links, 2 joints
Links:
- link upper_leg_front_left_link: geometry collision box size=.02 0.02 .12; visual box size=.02 0.02 .12
Joints:
- joint base_to_upper_leg_front_left: axis 0 0 1 -> 0 1 0; origin xyz=0.2 0.0 -0.1 rpy=0 0 0 -> xyz=0.113 0.08 -0.06 rpy=0.0 0.5 0
