Commit message: two link arm

File: urdf/two_link_arm.urdf (robot description, URDF)
Before this commit: robot omnipointer, 3 links, 2 joints
Links:
- added link arm_link_2, mass 0.29302326; collision box size=0.0356 0.05 0.317; visual box size=0.0356 0.05 0.317
- link arm_link_1: mass 0.190421352 -> 0.21931466; geometry collision box size=0.0356 0.05 0.202; visual box size=0.0356 0.05 0.202
Joints:
- removed joint base_to_link0
- removed joint link0_to_link1
- added joint arm_joint_0: type fixed, parent base_link, child arm_link_0, origin xyz=0 0 0.8 rpy=0 0 0
- added joint arm_joint_1: type revolute, parent arm_link_0, child arm_link_1, origin xyz=0 0 0.0545 rpy=0 0 0, axis 0 1 0, limit lower=-3.1415926535 upper=3.1415926535 effort=30.0 velocity=5.0
- added joint arm_joint_2: type revolute, parent arm_link_1, child arm_link_2, origin xyz=0 0 0.202 rpy=0 0 0, axis 0 1 0, limit lower=-1.57079632679 upper=1.57079632679 effort=30.0 velocity=5.0
