Commit message: add trajectory data

File: urdf/laikago/laikago.urdf (robot description, URDF)
Before this commit: robot plane, 13 links, 12 joints
Links:
- added link base_link, mass 0.1
Joints:
- added joint add_height_joint: type revolute, parent base_link, child chassis, origin xyz=0 0 0.5 rpy=0 0 0, axis 1 0 0, limit lower=-3.1415926535 upper=3.1415926535 effort=30.0 velocity=5.0

Commit message: quadrupedal render works

File: urdf/laikago/laikago.urdf (robot description, URDF)
Before this commit: robot plane, 14 links, 13 joints
Joints:
- joint FR_hip_motor_2_chassis_joint: axis 0 0 -1 -> 0 0 1
- joint RR_hip_motor_2_chassis_joint: axis 0 0 -1 -> 0 0 1
